File: nRF52810 Beacon/Rev1/nRF52810 Beacon.sch (EAGLE design)
At the start: 18 parts, among them IC1 NRF52810_QF48

Commit message: nrf52 revizeler
Parts:
- removed C16: 100nF, Nordic_nRF:CAPACITOR_0603_N
- removed U$1: SERIALWIRE, PoiLabs:SERIALWIRE
- added C28: 100nF, Nordic_misc:CAPACITOR_0603_N
Connections:
- new net ANT: L1.2
- net GND: now also C28.2; no longer C16.2, U$1.GND
- net SWDCLK: no longer U$1.SWDCLK
- net SWDIO: no longer U$1.SWDIO
- net VDD: now also C28.1; no longer C16.1, U$1.VDD
Other:
- note added: "Oğuzhan Memiş December 23 Rev1 nRF52810 Beacon Project 32 clock eklendi programlama pini revize edildi anten revize edildi"
- note removed: "Oğuzhan Memiş December 23 Rev 0 nRF52810 Beacon Project"
- moved on the sheet: BT1
Changed lines of the file:
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@@
 <schematic_group name="32MHZ" style="continuous"/>
 <schematic_group name="BATTERY" style="continuous"/>
-<schematic_group name="PROGRAMMER" style="continuous" titleSize="1"/>
 </groups>
 <parts>
@@
 <part name="SUPPLY11" library="supply2" library_urn="urn:adsk.eagle:library:372" deviceset="GND" device=""/>
 <part name="SUPPLY12" library="supply2" library_urn="urn:adsk.eagle:library:372" deviceset="VDD" device=""/>
-<part name="U$1" library="PoiLabs" deviceset="SERIALWIRE" device=""/>
 <part name="BT1" library="2462" deviceset="2462" device=""/>
-<part name="C16" library="Nordic_nRF" library_urn="urn:adsk.eagle:library:169009" deviceset="CAPACITOR" device="_0603_N" package3d_urn="urn:adsk.eagle:package:2593734/1" value="100nF"/>
+<part name="C28" library="Nordic_misc" deviceset="CAPACITOR" device="_0603_N" value="100nF"/>
 </parts>
 <sheets>
@@
 <text x="169" y="-0.87" size="1.778" layer="91">Oğuzhan Memiş
 December 23
-Rev 0
-nRF52810 Beacon Project</text>
+Rev1
+nRF52810 Beacon Project
+32 clock eklendi
+programlama pini revize edildi
+anten revize edildi</text>
 <frame x1="35.7" y1="-11.5" x2="207" y2="130.1" columns="8" rows="5" layer="91"/>
 </plain>
@@
 <attribute name="VALUE" x="112.777" y="110.192" size="1.778" layer="96" rot="R180"/>
 </instance>
-<instance part="U$1" gate="G$1" x="60.85" y="21.85" smashed="yes" grouprefs="PROGRAMMER"/>
-<instance part="BT1" gate="G$1" x="59.45" y="2.95" smashed="yes" grouprefs="BATTERY">
-<attribute name="NAME" x="55.64" y="6.76" size="1.778" layer="95"/>
-<attribute name="VALUE" x="55.64" y="-2.13" size="1.778" layer="96"/>
-</instance>
-<instance part="C16" gate="C$1" x="57.9" y="43.9" smashed="yes" rot="R90" grouprefs="PROGRAMMER">
-<attribute name="NAME" x="61.276" y="47.919" size="1.778" layer="95" rot="R180"/>
+<instance part="BT1" gate="G$1" x="62.55" y="43.75" smashed="yes" grouprefs="BATTERY">
+<attribute name="NAME" x="58.74" y="47.56" size="1.778" layer="95"/>
+<attribute name="VALUE" x="58.74" y="38.67" size="1.778" layer="96"/>
+</instance>
+<instance part="C28" gate="C$1" x="60.4" y="17.8" smashed="yes" rot="R90">
+<attribute name="NAME" x="62.976" y="21.119" size="1" layer="95" rot="R180"/>
 </instance>
 </instances>
@@
 </segment>
 <segment>
-<pinref part="U$1" gate="G$1" pin="GND"/>
-<wire x1="63.39" y1="32.01" x2="63.39" y2="33.01" width="0.1524" layer="91" grouprefs="PROGRAMMER"/>
-<label x="63.35" y="33" size="1" layer="95" rot="R90" xref="yes" grouprefs="PROGRAMMER"/>
-<pinref part="C16" gate="C$1" pin="2"/>
-<wire x1="62.98" y1="43.9" x2="65.3" y2="43.9" width="0.1524" layer="91" grouprefs="PROGRAMMER"/>
-<wire x1="65.3" y1="43.9" x2="65.3" y2="32.01" width="0.1524" layer="91" grouprefs="PROGRAMMER"/>
-<wire x1="65.3" y1="32" x2="65.3" y2="32.01" width="0.1524" layer="91" grouprefs="PROGRAMMER"/>
-<wire x1="65.3" y1="32.01" x2="63.39" y2="32.01" width="0.1524" layer="91" grouprefs="PROGRAMMER"/>
-<junction x="63.39" y="32.01" grouprefs="PROGRAMMER"/>
-</segment>
-<segment>
 <pinref part="BT1" gate="G$1" pin="NEG"/>
-<wire x1="67.07" y1="2.95" x2="70" y2="2.95" width="0.1524" layer="91" grouprefs="BATTERY"/>
-<label x="69.9" y="2.85" size="1" layer="95" xref="yes" grouprefs="BATTERY"/>
+<wire x1="70.17" y1="43.75" x2="73.1" y2="43.75" width="0.1524" layer="91" grouprefs="BATTERY"/>
+<label x="73" y="43.65" size="1" layer="95" xref="yes" grouprefs="BATTERY"/>
 </segment>
 <segment>
@@
 <wire x1="60.884" y1="92.77919375" x2="60.884" y2="91.059" width="0.1524" layer="91"/>
 </segment>
+<segment>
+<pinref part="C28" gate="C$1" pin="2"/>
+<wire x1="65.48" y1="17.8" x2="69.7" y2="17.8" width="0.1524" layer="91"/>
+<label x="69.8" y="17.8" size="1" layer="95" rot="R90" xref="yes"/>
+</segment>
 </net>
 <net name="VDD" class="0">
@@
 </segment>
 <segment>
-<pinref part="U$1" gate="G$1" pin="VDD"/>
-<wire x1="55.77" y1="32.01" x2="55.77" y2="33.3" width="0.1524" layer="91" grouprefs="PROGRAMMER"/>
-<label x="55.75" y="33.25" size="1" layer="95" rot="R90" xref="yes" grouprefs="PROGRAMMER"/>
-<wire x1="55.77" y1="32.01" x2="52.5" y2="32.01" width="0.1524" layer="91" grouprefs="PROGRAMMER"/>
-<wire x1="52.5" y1="32.01" x2="52.5" y2="43.9" width="0.1524" layer="91" grouprefs="PROGRAMMER"/>
-<junction x="55.77" y="32.01" grouprefs="PROGRAMMER"/>
-<pinref part="C16" gate="C$1" pin="1"/>
-<wire x1="52.5" y1="43.9" x2="55.36" y2="43.9" width="0.1524" layer="91" grouprefs="PROGRAMMER"/>
-</segment>
-<segment>
 <pinref part="BT1" gate="G$1" pin="POS"/>
-<wire x1="51.83" y1="2.95" x2="48.83" y2="2.95" width="0.1524" layer="91" grouprefs="BATTERY"/>
-<label x="48.85" y="2.95" size="1" layer="95" rot="R180" xref="yes" grouprefs="BATTERY"/>
+<wire x1="54.93" y1="43.75" x2="51.93" y2="43.75" width="0.1524" layer="91" grouprefs="BATTERY"/>
+<label x="51.95" y="43.75" size="1" layer="95" rot="R180" xref="yes" grouprefs="BATTERY"/>
 </segment>
 <segment>
@@
 <junction x="114.24" y="104"/>
 </segment>
+<segment>
+<pinref part="C28" gate="C$1" pin="1"/>
+<wire x1="57.86" y1="17.8" x2="54.5" y2="17.8" width="0.1524" layer="91"/>
+<label x="54.5" y="17.9" size="1" layer="95" rot="R90" xref="yes"/>
+</segment>
 </net>
 <net name="SWDIO" class="0">
@@
 <label x="170.297" y="50.18" size="1" layer="95" rot="R270" xref="yes"/>
 </segment>
-<segment>
-<pinref part="U$1" gate="G$1" pin="SWDIO"/>
-<wire x1="58.31" y1="32.01" x2="58.31" y2="33.01" width="0.1524" layer="91" grouprefs="PROGRAMMER"/>
-<label x="58.3" y="33.1" size="1" layer="95" rot="R90" xref="yes" grouprefs="PROGRAMMER"/>
-</segment>
 </net>
 <net name="SWDCLK" class="0">
@@
 <wire x1="167.706" y1="55.729" x2="167.694" y2="50.171" width="0.1524" layer="91"/>
 <label x="167.68" y="50.171" size="1" layer="95" rot="R270" xref="yes"/>
-</segment>
-<segment>
-<pinref part="U$1" gate="G$1" pin="SWDCLK"/>
-<wire x1="60.85" y1="32.01" x2="60.85" y2="33.01" width="0.1524" layer="91" grouprefs="PROGRAMMER"/>
-<label x="60.9" y="33.05" size="1" layer="95" rot="R90" xref="yes" grouprefs="PROGRAMMER"/>
 </segment>
 </net>
@@
 </segment>
 </net>
+<net name="ANT" class="0">
+<segment>
+<pinref part="L1" gate="L$1" pin="2"/>
+<wire x1="195.491" y1="68.432" x2="198.6" y2="68.432" width="0.1524" layer="91"/>
+<wire x1="198.6" y1="68.432" x2="198.6" y2="68.4" width="0.1524" layer="91"/>
+<label x="198.6" y="68.4" size="2" layer="95" rot="R90" xref="yes"/>
+</segment>
+</net>
